Commit message: Added ZED cameras to Gazebo

File: swerve_description/urdf/swerve.xacro (robot description, xacro)
@@ -162,5 +162,5 @@
       <parent link="zed_center"/>
       <child link="zed_left_camera"/>
-      <origin xyz="0.2 0.06 0" rpy="0 0 0" />
+      <origin xyz="0 0.06 0" rpy="0 0 0" />
     </joint>
     <joint name="zed_right_camera_joint" type="fixed">

File: swerve_description/urdf/swerve_gazebo.xacro (robot description, xacro)
@@ -67,5 +67,100 @@
     ZED CAMERA
   -->
-  <gazebo reference="zed_left_camera">
+  <gazebo reference="zed_center">
+    <sensor type="multicamera" name="zed_camera">
+      <update_rate>30.0</update_rate>
+      <camera name="zed_left_camera">
+        <pose>0 0.06 0 0 0 0</pose>
+        <horizontal_fov>0.8709216071359963</horizontal_fov>
+        <image>
+          <width>640</width>
+          <height>480</height>
+          <format>R8G8B8</format>
+        </image>
+        <clip>
+          <near>0.5</near>
+          <far>20</far>
+        </clip>
+        <noise>
+          <type>gaussian</type>
+          <mean>0.0</mean>
+          <stddev>0.007</stddev>
+        </noise>
+      </camera>
+      <camera name="zed_right_camera">
+        <pose>0 -0.06 0 0 0 0</pose>
+        <horizontal_fov>0.8709216071359963</horizontal_fov>
+        <image>
+          <width>640</width>
+          <height>480</height>
+          <format>R8G8B8</format>
+        </image>
+        <clip>
+          <near>0.5</near>
+          <far>20</far>
+        </clip>
+        <noise>
+          <type>gaussian</type>
+          <mean>0.0</mean>
+          <stddev>0.007</stddev>
+        </noise>
+      </camera>
+      <plugin name="stereo_camera_controller" filename="libgazebo_ros_multicamera.so">
+        <alwaysOn>true</alwaysOn>
+        <updateRate>0.0</updateRate>
+        <cameraName>camera</cameraName>
+        <imageTopicName>image_raw_color</imageTopicName>
+        <cameraInfoTopicName>camera_info</cameraInfoTopicName>
+        <frameName>zed_center</frameName>
+        <hackBaseline>0</hackBaseline>
+        <distortionK1>0.0</distortionK1>
+        <distortionK2>0.0</distortionK2>
+        <distortionK3>0.0</distortionK3>
+        <distortionT1>0.0</distortionT1>
+        <distortionT2>0.0</distortionT2>
+      </plugin>
+    </sensor>
+  </gazebo>
+  <!-- <gazebo>
+    <sensor type="camera" name="left_camera">
+      <update_rate>30.0</update_rate>
+      <camera>
+        <horizontal_fov>2.0</horizontal_fov>
+        <image>
+          <width>800</width>
+          <height>800</height>
+          <format>R8G8B8</format>
+        </image>
+        <clip>
+          <near>0.02</near>
+          <far>300</far>
+        </clip>
+      </camera>
+    <plugin name="depth_camera_controller" filename="libgazebo_ros_openni_kinect.so">
+      <baseline>0.2</baseline>
+      <alwaysOn>true</alwaysOn>
+      <updateRate>0</updateRate>
+      <cameraName>zed_camera</cameraName>
+      <imageTopicName>/camera/depth/image_raw</imageTopicName>
+      <cameraInfoTopicName>/camera/depth/camera_info</cameraInfoTopicName>
+      <depthImageTopicName>/camera/depth/image_raw</depthImageTopicName>
+      <depthImageInfoTopicName>/camera/depth/camera_info</depthImageInfoTopicName>
+      <pointCloudTopicName>/camera/depth/points</pointCloudTopicName>
+      <frameName>zed_center</frameName>
+      <pointCloudCutoff>0.5</pointCloudCutoff>
+      <distortionK1>0.00000001</distortionK1>
+      <distortionK2>0.00000001</distortionK2>
+      <distortionK3>0.00000001</distortionK3>
+      <distortionT1>0.00000001</distortionT1>
+      <distortionT2>0.00000001</distortionT2>
+      <CxPrime>0</CxPrime>
+      <Cx>0</Cx>
+      <Cy>0</Cy>
+      <focalLength>0</focalLength>
+      <hackBaseline>0</hackBaseline>
+    </plugin>
+    </sensor>
+  </gazebo> -->
+  <!-- <gazebo reference="zed_left_camera">
     <material>Gazebo/Green</material>
     <sensor type="camera" name="left_camera">
@@ -98,5 +193,5 @@
       </plugin>
     </sensor>
-  </gazebo>
+  </gazebo> -->
   <!-- <gazebo reference="zed_left_camera">
     <sensor type="camera" name="zed_left_camera">
@@ -171,58 +266,3 @@
     </sensor>
   </gazebo> -->
-  <!-- <gazebo reference="zed_center">
-    <sensor type="multicamera" name="zed_camera">
-      <update_rate>30.0</update_rate>
-      <camera name="zed_left_camera">
-        <pose>0 0.06 0 0 0 0</pose>
-        <horizontal_fov>0.8709216071359963</horizontal_fov>
-        <image>
-          <width>640</width>
-          <height>480</height>
-          <format>R8G8B8</format>
-        </image>
-        <clip>
-          <near>0.02</near>
-          <far>300</far>
-        </clip>
-        <noise>
-          <type>gaussian</type>
-          <mean>0.0</mean>
-          <stddev>0.007</stddev>
-        </noise>
-      </camera>
-      <camera name="zed_right_camera">
-        <pose>0 -0.06 0 0 0 0</pose>
-        <horizontal_fov>0.8709216071359963</horizontal_fov>
-        <image>
-          <width>640</width>
-          <height>480</height>
-          <format>R8G8B8</format>
-        </image>
-        <clip>
-          <near>0.02</near>
-          <far>300</far>
-        </clip>
-        <noise>
-          <type>gaussian</type>
-          <mean>0.0</mean>
-          <stddev>0.007</stddev>
-        </noise>
-      </camera>
-      <plugin name="stereo_camera_controller" filename="libgazebo_ros_multicamera.so">
-        <alwaysOn>true</alwaysOn>
-        <updateRate>0.0</updateRate>
-        <cameraName>camera</cameraName>
-        <imageTopicName>image_raw_color</imageTopicName>
-        <cameraInfoTopicName>camera_info</cameraInfoTopicName>
-        <frameName>zed_center</frameName>
-        <hackBaseline>0</hackBaseline>
-        <distortionK1>0.0</distortionK1>
-        <distortionK2>0.0</distortionK2>
-        <distortionK3>0.0</distortionK3>
-        <distortionT1>0.0</distortionT1>
-        <distortionT2>0.0</distortionT2>
-      </plugin>
-    </sensor>
-  </gazebo> -->
 </robot>

Commit message: Added depth camera to Swerve
Need to test on a computer with OpenGL

File: swerve_description/urdf/swerve.xacro (robot description, xacro)
@@ -34,22 +34,22 @@
     <xacro:swerve_joint joint_name="${name}_joint_FS" parent="${name}_body" child="${name}_FS_link"
       x="0" y="0.381" hardware_interface="${hardware_interface}"/>
-      <link name="${name}_FS_link">
+    <link name="${name}_FS_link">
+      <inertial>
+        <origin xyz="-5.819E-13 -0.062713 0" rpy="0 0 0" />
+        <mass value="${swivel_mass}" />
+        <inertia ixx="0.0010313" ixy="1.377E-13" ixz="4.6213E-21" iyy="0.00038801" iyz="-9.7714E-21" izz="0.001103" />
+      </inertial>
+      <xacro:insert_block name="swivel_visual_collision" />
+    </link>
+    <xacro:wheel_joint joint_name="${name}_joint_FW" parent="${name}_FS_link" child="${name}_FW_link"
+      hardware_interface="${hardware_interface}"/>
+      <link name="${name}_FW_link">
         <inertial>
-          <origin xyz="-5.819E-13 -0.062713 0" rpy="0 0 0" />
-          <mass value="${swivel_mass}" />
-          <inertia ixx="0.0010313" ixy="1.377E-13" ixz="4.6213E-21" iyy="0.00038801" iyz="-9.7714E-21" izz="0.001103" />
+          <origin xyz="-7.8185E-19 2.7756E-17 5.5511E-17" rpy="0 0 0" />
+          <mass value="${wheel_mass}" />
+          <inertia ixx="0.00016727" ixy="-4.9394E-22" ixz="-2.3462E-22" iyy="9.626E-05" iyz="-1.4682E-20" izz="9.626E-05" />
         </inertial>
-        <xacro:insert_block name="swivel_visual_collision" />
+        <xacro:insert_block name="wheel_visual_collision" />
       </link>
-      <xacro:wheel_joint joint_name="${name}_joint_FW" parent="${name}_FS_link" child="${name}_FW_link"
-        hardware_interface="${hardware_interface}"/>
-        <link name="${name}_FW_link">
-          <inertial>
-            <origin xyz="-7.8185E-19 2.7756E-17 5.5511E-17" rpy="0 0 0" />
-            <mass value="${wheel_mass}" />
-            <inertia ixx="0.00016727" ixy="-4.9394E-22" ixz="-2.3462E-22" iyy="9.626E-05" iyz="-1.4682E-20" izz="9.626E-05" />
-          </inertial>
-          <xacro:insert_block name="wheel_visual_collision" />
-        </link>
     <!--
       LEFT SWIVEL DEFINITION
@@ -57,22 +57,22 @@
     <xacro:swerve_joint joint_name="${name}_joint_LS" parent="${name}_body" child="${name}_LS_link"
       x="-0.32996" y="-0.1905" hardware_interface="${hardware_interface}"/>
-      <link name="${name}_LS_link">
+    <link name="${name}_LS_link">
+      <inertial>
+        <origin xyz="-5.8187E-13 -0.062713 0" rpy="0 0 0" />
+        <mass value="${swivel_mass}" />
+        <inertia ixx="0.0010313" ixy="1.377E-13" ixz="1.6475E-20" iyy="0.00038801" iyz="2.1123E-20" izz="0.001103" />
+      </inertial>
+      <xacro:insert_block name="swivel_visual_collision" />
+    </link>
+    <xacro:wheel_joint joint_name="${name}_joint_LW" parent="${name}_LS_link" child="${name}_LW_link"
+      hardware_interface="${hardware_interface}"/>
+      <link name="${name}_LW_link">
         <inertial>
-          <origin xyz="-5.8187E-13 -0.062713 0" rpy="0 0 0" />
-          <mass value="${swivel_mass}" />
-          <inertia ixx="0.0010313" ixy="1.377E-13" ixz="1.6475E-20" iyy="0.00038801" iyz="2.1123E-20" izz="0.001103" />
+          <origin xyz="0 2.7756E-17 0" rpy="0 0 0" />
+          <mass value="${wheel_mass}" />
+          <inertia ixx="0.00016727" ixy="-1.3787E-22" ixz="-1.031E-22" iyy="9.626E-05" iyz="-3.3087E-21" izz="9.626E-05" />
         </inertial>
-        <xacro:insert_block name="swivel_visual_collision" />
+        <xacro:insert_block name="wheel_visual_collision" />
       </link>
-      <xacro:wheel_joint joint_name="${name}_joint_LW" parent="${name}_LS_link" child="${name}_LW_link"
-        hardware_interface="${hardware_interface}"/>
-        <link name="${name}_LW_link">
-          <inertial>
-            <origin xyz="0 2.7756E-17 0" rpy="0 0 0" />
-            <mass value="${wheel_mass}" />
-            <inertia ixx="0.00016727" ixy="-1.3787E-22" ixz="-1.031E-22" iyy="9.626E-05" iyz="-3.3087E-21" izz="9.626E-05" />
-          </inertial>
-          <xacro:insert_block name="wheel_visual_collision" />
-        </link>
     <!--
       RIGHT SWIVEL DEFINITION
@@ -80,22 +80,22 @@
     <xacro:swerve_joint joint_name="${name}_joint_RS" parent="${name}_body" child="${name}_RS_link"
       x="0.32996" y="-0.1905"  hardware_interface="${hardware_interface}"/>
-      <link name="${name}_RS_link">
+    <link name="${name}_RS_link">
+      <inertial>
+        <origin xyz="-5.8192E-13 -0.062713 -2.7756E-17" rpy="0 0 0" />
+        <mass value="${swivel_mass}" />
+        <inertia ixx="0.0010313" ixy="1.377E-13" ixz="1.6475E-20" iyy="0.00038801" iyz="2.1123E-20" izz="0.001103" />
+      </inertial>
+      <xacro:insert_block name="swivel_visual_collision" />
+    </link>
+    <xacro:wheel_joint joint_name="${name}_joint_RW" parent="${name}_RS_link" child="${name}_RW_link"
+      hardware_interface="${hardware_interface}"/>
+      <link name="${name}_RW_link">
         <inertial>
-          <origin xyz="-5.8192E-13 -0.062713 -2.7756E-17" rpy="0 0 0" />
-          <mass value="${swivel_mass}" />
-          <inertia ixx="0.0010313" ixy="1.377E-13" ixz="1.6475E-20" iyy="0.00038801" iyz="2.1123E-20" izz="0.001103" />
+          <origin xyz="-5.5511E-17 2.7756E-17 -2.7756E-17" rpy="0 0 0" />
+          <mass value="${wheel_mass}" />
+          <inertia ixx="0.00016727" ixy="-1.3787E-22" ixz="-1.031E-22" iyy="9.626E-05" iyz="-3.3087E-21" izz="9.626E-05" />
         </inertial>
-        <xacro:insert_block name="swivel_visual_collision" />
+        <xacro:insert_block name="wheel_visual_collision" />
       </link>
-      <xacro:wheel_joint joint_name="${name}_joint_RW" parent="${name}_RS_link" child="${name}_RW_link"
-        hardware_interface="${hardware_interface}"/>
-        <link name="${name}_RW_link">
-          <inertial>
-            <origin xyz="-5.5511E-17 2.7756E-17 -2.7756E-17" rpy="0 0 0" />
-            <mass value="${wheel_mass}" />
-            <inertia ixx="0.00016727" ixy="-1.3787E-22" ixz="-1.031E-22" iyy="9.626E-05" iyz="-3.3087E-21" izz="9.626E-05" />
-          </inertial>
-          <xacro:insert_block name="wheel_visual_collision" />
-        </link>
     <!--
       SENSORS
@@ -136,4 +136,10 @@
       <child link="zed_center"/>
       <origin xyz="0 0.18 0.11" rpy="0 0 ${pi}" />
+    </joint>
+    <link name="zed_depth"></link>
+    <joint name="zed_depth_joint" type="fixed">
+      <parent link="zed_center"/>
+      <child link="zed_depth"/>
+      <origin xyz="0 0 0" rpy="${pi} 0 ${pi}" />
     </joint>
     <link name="zed_left_camera">

File: swerve_description/urdf/swerve_gazebo.xacro (robot description, xacro)
@@ -8,25 +8,25 @@
 <robot name="swerve" xmlns:xacro="http://www.ros.org/wiki/xacro">
   <!--
-    ODOM CONTROLLER
+  ODOM CONTROLLER
   -->
-	<gazebo>
-		<plugin name="gazebo_ros_controller" filename="libgazebo_ros_control.so">
-			<robotNamespace>/swerve</robotNamespace>
-		</plugin>
-		<plugin name="p3d_base_controller" filename="libgazebo_ros_p3d.so">
-			<alwaysOn>true</alwaysOn>
-			<updateRate>50.0</updateRate>
-			<bodyName>odom</bodyName>
-			<topicName>odom</topicName>
-			<gaussianNoise>0.01</gaussianNoise>
-			<frameName>world</frameName>
-			<xyzOffsets>0 0 0</xyzOffsets>
-			<rpyOffsets>0 0 0</rpyOffsets>
-		</plugin>
-	</gazebo>
+  <gazebo>
+    <plugin name="gazebo_ros_controller" filename="libgazebo_ros_control.so">
+      <robotNamespace>/swerve</robotNamespace>
+    </plugin>
+    <plugin name="p3d_base_controller" filename="libgazebo_ros_p3d.so">
+      <alwaysOn>true</alwaysOn>
+      <updateRate>50.0</updateRate>
+      <bodyName>odom</bodyName>
+      <topicName>odom</topicName>
+      <gaussianNoise>0.01</gaussianNoise>
+      <frameName>world</frameName>
+      <xyzOffsets>0 0 0</xyzOffsets>
+      <rpyOffsets>0 0 0</rpyOffsets>
+    </plugin>
+  </gazebo>
   <!--
-    LIDAR
+  LIDAR
   -->
-	<gazebo reference="laser">
+  <gazebo reference="laser">
     <sensor type="gpu_ray" name="laser">
       <always_on>true</always_on>
@@ -51,12 +51,12 @@
           <type>gaussian</type>
           <!-- Noise parameters based on published spec for Hokuyo laser
-               achieving "+-30mm" accuracy at range < 10m.  A mean of 0.0m and
-               stddev of 0.01m will put 99.7% of samples within 0.03m of the true
-               reading. -->
-          <mean>0.0</mean>
-          <stddev>0.01</stddev>
-        </noise>
-      </ray>
-      <plugin name="gazebo_ros_head_hokuyo_controller" filename="libgazebo_ros_gpu_laser.so">
+           achieving "+-30mm" accuracy at range < 10m.  A mean of 0.0m and
+           stddev of 0.01m will put 99.7% of samples within 0.03m of the true
+           reading. -->
+           <mean>0.0</mean>
+           <stddev>0.01</stddev>
+         </noise>
+       </ray>
+       <plugin name="gazebo_ros_head_hokuyo_controller" filename="libgazebo_ros_gpu_laser.so">
         <topicName>scan</topicName>
         <frameName>laser</frameName>
@@ -65,5 +65,5 @@
   </gazebo>
   <!--
-    ZED CAMERA
+  ZED CAMERA
   -->
   <gazebo reference="zed_center">
@@ -110,5 +110,5 @@
         <updateRate>0.0</updateRate>
         <cameraName>camera</cameraName>
-        <imageTopicName>image_raw_color</imageTopicName>
+        <imageTopicName>image_raw</imageTopicName>
         <cameraInfoTopicName>camera_info</cameraInfoTopicName>
         <frameName>zed_center</frameName>
@@ -122,147 +122,39 @@
     </sensor>
   </gazebo>
-  <!-- <gazebo>
-    <sensor type="camera" name="left_camera">
-      <update_rate>30.0</update_rate>
+  <gazebo reference="zed_depth">
+    <sensor type="depth" name="camera">
+      <always_on>true</always_on>
+      <update_rate>20.0</update_rate>
       <camera>
         <horizontal_fov>2.0</horizontal_fov>
         <image>
-          <width>800</width>
-          <height>800</height>
-          <format>R8G8B8</format>
+          <format>B8G8R8</format>
+          <width>640</width>
+          <height>480</height>
         </image>
         <clip>
-          <near>0.02</near>
-          <far>300</far>
+          <near>0.05</near>
+          <far>8.0</far>
         </clip>
       </camera>
-    <plugin name="depth_camera_controller" filename="libgazebo_ros_openni_kinect.so">
-      <baseline>0.2</baseline>
-      <alwaysOn>true</alwaysOn>
-      <updateRate>0</updateRate>
-      <cameraName>zed_camera</cameraName>
-      <imageTopicName>/camera/depth/image_raw</imageTopicName>
-      <cameraInfoTopicName>/camera/depth/camera_info</cameraInfoTopicName>
-      <depthImageTopicName>/camera/depth/image_raw</depthImageTopicName>
-      <depthImageInfoTopicName>/camera/depth/camera_info</depthImageInfoTopicName>
-      <pointCloudTopicName>/camera/depth/points</pointCloudTopicName>
-      <frameName>zed_center</frameName>
-      <pointCloudCutoff>0.5</pointCloudCutoff>
-      <distortionK1>0.00000001</distortionK1>
-      <distortionK2>0.00000001</distortionK2>
-      <distortionK3>0.00000001</distortionK3>
-      <distortionT1>0.00000001</distortionT1>
-      <distortionT2>0.00000001</distortionT2>
-      <CxPrime>0</CxPrime>
-      <Cx>0</Cx>
-      <Cy>0</Cy>
-      <focalLength>0</focalLength>
-      <hackBaseline>0</hackBaseline>
-    </plugin>
-    </sensor>
-  </gazebo> -->
-  <!-- <gazebo reference="zed_left_camera">
-    <material>Gazebo/Green</material>
-    <sensor type="camera" name="left_camera">
-      <update_rate>30.0</update_rate>
-      <camera name="left">
-        <horizontal_fov>2.0</horizontal_fov>
-        <image>
-          <width>800</width>
-          <height>800</height>
-          <format>R8G8B8</format>
-        </image>
-        <clip>
-          <near>0.02</near>
-          <far>300</far>
-        </clip>
-      </camera>
-      <plugin name="camera_controller" filename="libgazebo_ros_camera.so">
+      <plugin name="kinect_camera_controller" filename="libgazebo_ros_openni_kinect.so">
+        <cameraName>camera</cameraName>
         <alwaysOn>true</alwaysOn>
-        <updateRate>0.0</updateRate>
-        <cameraName>camera/left</cameraName>
-        <imageTopicName>image_raw</imageTopicName>
-        <cameraInfoTopicName>camera_info</cameraInfoTopicName>
-        <frameName>zed_left_camera</frameName>
-        <hackBaseline>0.07</hackBaseline>
-        <distortionK1>0.0</distortionK1>
-        <distortionK2>0.0</distortionK2>
-        <distortionK3>0.0</distortionK3>
-        <distortionT1>0.0</distortionT1>
-        <distortionT2>0.0</distortionT2>
+        <updateRate>10</updateRate>
+        <imageTopicName>rgb/image_raw</imageTopicName>
+        <depthImageTopicName>depth/image_raw</depthImageTopicName>
+        <pointCloudTopicName>depth/points</pointCloudTopicName>
+        <cameraInfoTopicName>rgb/camera_info</cameraInfoTopicName>
+        <depthImageCameraInfoTopicName>depth/camera_info</depthImageCameraInfoTopicName>
+        <frameName>zed_depth</frameName>
+        <baseline>0.1</baseline>
+        <distortion_k1>0.0</distortion_k1>
+        <distortion_k2>0.0</distortion_k2>
+        <distortion_k3>0.0</distortion_k3>
+        <distortion_t1>0.0</distortion_t1>
+        <distortion_t2>0.0</distortion_t2>
+        <pointCloudCutoff>0.4</pointCloudCutoff>
       </plugin>
     </sensor>
-  </gazebo> -->
-  <!-- <gazebo reference="zed_left_camera">
-    <sensor type="camera" name="zed_left_camera">
-      <update_rate>30.0</update_rate>
-      <camera name="zed_left_camera">
-        <horizontal_fov>0.8709216071359963</horizontal_fov>
-        <image>
-          <width>640</width>
-          <height>480</height>
-          <format>B8G8R8</format>
-        </image>
-        <clip>
-          <near>0.02</near>
-          <far>300</far>
-        </clip>
-        <noise>
-          <type>gaussian</type>
-          <mean>0.0</mean>
-          <stddev>0.007</stddev>
-        </noise>
-      </camera>
-      <plugin name="camera_controller" filename="libgazebo_ros_camera.so">
-        <alwaysOn>true</alwaysOn>
-        <updateRate>30.0</updateRate>
-        <cameraName>/camera/left</cameraName>
-        <imageTopicName>image_raw_color</imageTopicName>
-        <cameraInfoTopicName>camera_info</cameraInfoTopicName>
-        <frameName>zed_left_camera</frameName>
-        <hackBaseline>0</hackBaseline>
-        <distortionK1>0.0</distortionK1>
-        <distortionK2>0.0</distortionK2>
-        <distortionK3>0.0</distortionK3>
-        <distortionT1>0.0</distortionT1>
-        <distortionT2>0.0</distortionT2>
-      </plugin>
-    </sensor>
-  </gazebo> -->
-  <!-- <gazebo reference="zed_right_camera">
-    <sensor type="camera" name="zed_right_camera">
-      <update_rate>30.0</update_rate>
-      <camera name="zed_right_camera">
-        <horizontal_fov>0.8709216071359963</horizontal_fov>
-        <image>
-          <width>640</width>
-          <height>480</height>
-          <format>B8G8R8</format>
-        </image>
-        <clip>
-          <near>0.02</near>
-          <far>300</far>
-        </clip>
-        <noise>
-          <type>gaussian</type>
-          <mean>0.0</mean>
-          <stddev>0.007</stddev>
-        </noise>
-      </camera>
-      <plugin name="camera_controller" filename="libgazebo_ros_camera.so">
-        <alwaysOn>true</alwaysOn>
-        <updateRate>30.0</updateRate>
-        <cameraName>/camera/right</cameraName>
-        <imageTopicName>image_raw_color</imageTopicName>
-        <cameraInfoTopicName>camera_info</cameraInfoTopicName>
-        <frameName>zed_right_camera</frameName>
-        <hackBaseline>0</hackBaseline>
-        <distortionK1>0.0</distortionK1>
-        <distortionK2>0.0</distortionK2>
-        <distortionK3>0.0</distortionK3>
-        <distortionT1>0.0</distortionT1>
-        <distortionT2>0.0</distortionT2>
-      </plugin>
-    </sensor>
-  </gazebo> -->
+  </gazebo>
 </robot>
