Commit message: Interfaced Swerve in Gazebo with ROS

File: swerve_description/urdf/swerve.urdf.xacro (robot description, xacro)
@@ -12,4 +12,6 @@
   <!-- Import constants and modeling macros -->
   <xacro:include filename="$(find swerve_description)/urdf/swerve_utilities.xacro"/>
+  <!-- Import Gazebo tags -->
+  <xacro:include filename="$(find swerve_description)/urdf/swerve_gazebo.xacro"/>
   <!-- Import swerve robot -->
   <xacro:include filename="$(find swerve_description)/urdf/swerve.xacro"/>

File: swerve_description/urdf/swerve.xacro (robot description, xacro)
@@ -32,10 +32,5 @@
       FRONT SWIVEL DEFINITION
     -->
-    <joint name="${name}_joint_FS" type="continuous">
-      <origin xyz="0 0.381 0" rpy="1.5708 0 0" />
-      <parent link="${name}_body" />
-      <child link="${name}_FS_link" />
-      <axis xyz="0 -1 0" />
-    </joint>
+    <xacro:swerve_joint joint_name="${name}_joint_FS" parent="${name}_body" child="${name}_FS_link" x="0" y="0.381" />
     <link name="${name}_FS_link">
       <inertial>
@@ -58,10 +53,5 @@
       LEFT SWIVEL DEFINITION
     -->
-    <joint name="${name}_joint_LS" type="continuous">
-      <origin xyz="-0.32996 -0.1905 0" rpy="1.5708 0 0" />
-      <parent link="${name}_body" />
-      <child link="${name}_LS_link" />
-      <axis xyz="0 -1 0" />
-    </joint>
+    <xacro:swerve_joint joint_name="${name}_joint_LS" parent="${name}_body" child="${name}_LS_link" x="-0.32996" y="-0.1905" />
     <link name="${name}_LS_link">
       <inertial>
@@ -84,10 +74,5 @@
       RIGHT SWIVEL DEFINITION
     -->
-    <joint name="${name}_joint_RS" type="continuous">
-      <origin xyz="0.32996 -0.1905 0" rpy="1.5708 0 0" />
-      <parent link="${name}_body" />
-      <child link="${name}_RS_link" />
-      <axis xyz="0 -1 0" />
-    </joint>
+    <xacro:swerve_joint joint_name="${name}_joint_RS" parent="${name}_body" child="${name}_RS_link" x="0.32996" y="-0.1905" />
     <link name="${name}_RS_link">
       <inertial>

File: swerve_description/urdf/swerve_utilities.xacro (robot description, xacro)
@@ -7,4 +7,10 @@
 -->
 <robot name="swerve" xmlns:xacro="http://www.ros.org/wiki/xacro">
+  <!-- Constants -->
+  <xacro:property name="chassis_mass" value="7.0052" />
+  <xacro:property name="swivel_mass" value="0.449039" />
+  <xacro:property name="wheel_mass" value="0.15026" />
+  <xacro:property name="hardware_interface" value="PositionJointInterface" />
+  <xacro:property name="mechanical_reduction" value="1" />
   <!-- Common geometry properties -->
   <xacro:property name="chassis_geometry">
@@ -81,8 +87,32 @@
       <axis xyz="-1 0 0" />
     </joint>
+    <transmission name="${joint_name}_trans">
+      <type>transmission_interface/SimpleTransmission</type>
+      <joint name="${joint_name}">
+        <hardwareInterface>${hardware_interface}</hardwareInterface>
+      </joint>
+      <actuator name="${joint_name}_motor">
+        <mechanicalReduction>${mechanical_reduction}</mechanicalReduction>
+        <hardwareInterface>${hardware_interface}</hardwareInterface>
+      </actuator>
+    </transmission>
   </xacro:macro>
-  <!-- Constants -->
-  <xacro:property name="chassis_mass" value="7.0052" />
-  <xacro:property name="swivel_mass" value="0.449039" />
-  <xacro:property name="wheel_mass" value="0.15026" />
+  <xacro:macro name="swerve_joint" params="joint_name parent child x y">
+    <joint name="${joint_name}" type="continuous">
+      <origin xyz="${x} ${y} 0" rpy="1.5708 0 0" />
+      <parent link="${parent}" />
+      <child link="${child}" />
+      <axis xyz="0 -1 0" />
+    </joint>
+    <transmission name="${joint_name}_trans">
+      <type>transmission_interface/SimpleTransmission</type>
+      <joint name="${joint_name}">
+        <hardwareInterface>${hardware_interface}</hardwareInterface>
+      </joint>
+      <actuator name="${joint_name}_motor">
+        <mechanicalReduction>${mechanical_reduction}</mechanicalReduction>
+        <hardwareInterface>${hardware_interface}</hardwareInterface>
+      </actuator>
+    </transmission>
+  </xacro:macro>
 </robot>

Commit message: Added Swerve Navigation ROS package and odometry to Swerve in Gazebo

File: swerve_description/urdf/swerve.urdf.xacro (robot description, xacro)
@@ -7,4 +7,9 @@
 -->
 <robot name="swerve" xmlns:xacro="http://www.ros.org/wiki/xacro">
+  <!--
+    FIXED FRAME DEFINITION
+  -->
+  <!-- Fixed swerve dummy frame -->
+  <link name="odom" />
   <!--
     IMPORTS
@@ -17,13 +22,8 @@
   <xacro:include filename="$(find swerve_description)/urdf/swerve.xacro"/>
   <!--
-    WORLD DEFINITION
-  -->
-  <!-- Fixed dummy frame -->
-  <link name="swerve_base" />
-  <!--
     MACRO DEFINITIONS
   -->
   <!-- Define macros for swerve import -->
-  <xacro:swerve name="swerve" parent="swerve_base">
+  <xacro:swerve name="swerve" parent="odom" hardware_interface="$(arg hardware_interface)">
 	  <origin xyz="0 0 0.17" rpy="0 0 0"/>
   </xacro:swerve>

File: swerve_description/urdf/swerve.xacro (robot description, xacro)
@@ -9,5 +9,5 @@
   <!-- Include constants and modeling macros -->
   <xacro:include filename="$(find swerve_description)/urdf/swerve_utilities.xacro" />
-  <xacro:macro name="swerve" params="parent name *origin">
+  <xacro:macro name="swerve" params="parent name *origin hardware_interface">
     <!--
       DUMMY JOINT DEFINITION
@@ -32,5 +32,6 @@
       FRONT SWIVEL DEFINITION
     -->
-    <xacro:swerve_joint joint_name="${name}_joint_FS" parent="${name}_body" child="${name}_FS_link" x="0" y="0.381" />
+    <xacro:swerve_joint joint_name="${name}_joint_FS" parent="${name}_body" child="${name}_FS_link"
+        x="0" y="0.381" hardware_interface="${hardware_interface}"/>
     <link name="${name}_FS_link">
       <inertial>
@@ -41,5 +42,6 @@
       <xacro:insert_block name="swivel_visual_collision" />
     </link>
-    <xacro:wheel_joint joint_name="${name}_joint_FW" parent="${name}_FS_link" child="${name}_FW_link" />
+    <xacro:wheel_joint joint_name="${name}_joint_FW" parent="${name}_FS_link" child="${name}_FW_link"
+        hardware_interface="${hardware_interface}"/>
     <link name="${name}_FW_link">
       <inertial>
@@ -53,5 +55,6 @@
       LEFT SWIVEL DEFINITION
     -->
-    <xacro:swerve_joint joint_name="${name}_joint_LS" parent="${name}_body" child="${name}_LS_link" x="-0.32996" y="-0.1905" />
+    <xacro:swerve_joint joint_name="${name}_joint_LS" parent="${name}_body" child="${name}_LS_link"
+        x="-0.32996" y="-0.1905" hardware_interface="${hardware_interface}"/>
     <link name="${name}_LS_link">
       <inertial>
@@ -62,5 +65,6 @@
       <xacro:insert_block name="swivel_visual_collision" />
     </link>
-    <xacro:wheel_joint joint_name="${name}_joint_LW" parent="${name}_LS_link" child="${name}_LW_link" />
+    <xacro:wheel_joint joint_name="${name}_joint_LW" parent="${name}_LS_link" child="${name}_LW_link"
+        hardware_interface="${hardware_interface}"/>
     <link name="${name}_LW_link">
       <inertial>
@@ -74,5 +78,6 @@
       RIGHT SWIVEL DEFINITION
     -->
-    <xacro:swerve_joint joint_name="${name}_joint_RS" parent="${name}_body" child="${name}_RS_link" x="0.32996" y="-0.1905" />
+    <xacro:swerve_joint joint_name="${name}_joint_RS" parent="${name}_body" child="${name}_RS_link"
+        x="0.32996" y="-0.1905"  hardware_interface="${hardware_interface}"/>
     <link name="${name}_RS_link">
       <inertial>
@@ -83,5 +88,6 @@
       <xacro:insert_block name="swivel_visual_collision" />
     </link>
-    <xacro:wheel_joint joint_name="${name}_joint_RW" parent="${name}_RS_link" child="${name}_RW_link" />
+    <xacro:wheel_joint joint_name="${name}_joint_RW" parent="${name}_RS_link" child="${name}_RW_link"
+        hardware_interface="${hardware_interface}"/>
     <link name="${name}_RW_link">
       <inertial>

File: swerve_description/urdf/swerve_gazebo.xacro (robot description, xacro)
@@ -11,4 +11,14 @@
       <robotNamespace>/swerve</robotNamespace>
     </plugin>
+    <plugin name="p3d_base_controller" filename="libgazebo_ros_p3d.so">
+		  <alwaysOn>true</alwaysOn>
+		  <updateRate>50.0</updateRate>
+		  <bodyName>odom</bodyName>
+		  <topicName>odom</topicName>
+		  <gaussianNoise>0.01</gaussianNoise>
+		  <frameName>world</frameName>
+		  <xyzOffsets>0 0 0</xyzOffsets>
+		  <rpyOffsets>0 0 0</rpyOffsets>
+		</plugin>
   </gazebo>
 </robot>

File: swerve_description/urdf/swerve_utilities.xacro (robot description, xacro)
@@ -11,5 +11,4 @@
   <xacro:property name="swivel_mass" value="0.449039" />
   <xacro:property name="wheel_mass" value="0.15026" />
-  <xacro:property name="hardware_interface" value="PositionJointInterface" />
   <xacro:property name="mechanical_reduction" value="1" />
   <!-- Common geometry properties -->
@@ -80,5 +79,5 @@
   </xacro:property>
   <!-- Common joint properties -->
-  <xacro:macro name="wheel_joint" params="joint_name parent child">
+  <xacro:macro name="wheel_joint" params="joint_name parent child hardware_interface">
     <joint name="${joint_name}" type="continuous">
       <origin xyz="0 -0.127 0" rpy="0 0 0" />
@@ -98,5 +97,5 @@
     </transmission>
   </xacro:macro>
-  <xacro:macro name="swerve_joint" params="joint_name parent child x y">
+  <xacro:macro name="swerve_joint" params="joint_name parent child x y hardware_interface">
     <joint name="${joint_name}" type="continuous">
       <origin xyz="${x} ${y} 0" rpy="1.5708 0 0" />
