Commit message: Attempting cameas in Gazebo

File: swerve_description/urdf/swerve.urdf.xacro (robot description, xacro)
@@ -26,5 +26,5 @@
   <!-- Define macros for swerve import -->
   <xacro:swerve name="swerve" parent="odom" hardware_interface="$(arg hardware_interface)">
-	  <origin xyz="0 0 0.17" rpy="0 0 0"/>
+	  <origin xyz="0 0 0.17" rpy="0 0 -${pi}"/> <!-- rotate 90 degrees due to error in black box model -->
   </xacro:swerve>
 </robot>

File: swerve_description/urdf/swerve.xacro (robot description, xacro)
@@ -33,69 +33,146 @@
     -->
     <xacro:swerve_joint joint_name="${name}_joint_FS" parent="${name}_body" child="${name}_FS_link"
-        x="0" y="0.381" hardware_interface="${hardware_interface}"/>
-    <link name="${name}_FS_link">
-      <inertial>
-        <origin xyz="-5.819E-13 -0.062713 0" rpy="0 0 0" />
-        <mass value="${swivel_mass}" />
-        <inertia ixx="0.0010313" ixy="1.377E-13" ixz="4.6213E-21" iyy="0.00038801" iyz="-9.7714E-21" izz="0.001103" />
-      </inertial>
-      <xacro:insert_block name="swivel_visual_collision" />
-    </link>
-    <xacro:wheel_joint joint_name="${name}_joint_FW" parent="${name}_FS_link" child="${name}_FW_link"
+      x="0" y="0.381" hardware_interface="${hardware_interface}"/>
+      <link name="${name}_FS_link">
+        <inertial>
+          <origin xyz="-5.819E-13 -0.062713 0" rpy="0 0 0" />
+          <mass value="${swivel_mass}" />
+          <inertia ixx="0.0010313" ixy="1.377E-13" ixz="4.6213E-21" iyy="0.00038801" iyz="-9.7714E-21" izz="0.001103" />
+        </inertial>
+        <xacro:insert_block name="swivel_visual_collision" />
+      </link>
+      <xacro:wheel_joint joint_name="${name}_joint_FW" parent="${name}_FS_link" child="${name}_FW_link"
         hardware_interface="${hardware_interface}"/>
-    <link name="${name}_FW_link">
-      <inertial>
-        <origin xyz="-7.8185E-19 2.7756E-17 5.5511E-17" rpy="0 0 0" />
-        <mass value="${wheel_mass}" />
-        <inertia ixx="0.00016727" ixy="-4.9394E-22" ixz="-2.3462E-22" iyy="9.626E-05" iyz="-1.4682E-20" izz="9.626E-05" />
-      </inertial>
-      <xacro:insert_block name="wheel_visual_collision" />
-    </link>
+        <link name="${name}_FW_link">
+          <inertial>
+            <origin xyz="-7.8185E-19 2.7756E-17 5.5511E-17" rpy="0 0 0" />
+            <mass value="${wheel_mass}" />
+            <inertia ixx="0.00016727" ixy="-4.9394E-22" ixz="-2.3462E-22" iyy="9.626E-05" iyz="-1.4682E-20" izz="9.626E-05" />
+          </inertial>
+          <xacro:insert_block name="wheel_visual_collision" />
+        </link>
     <!--
       LEFT SWIVEL DEFINITION
     -->
     <xacro:swerve_joint joint_name="${name}_joint_LS" parent="${name}_body" child="${name}_LS_link"
-        x="-0.32996" y="-0.1905" hardware_interface="${hardware_interface}"/>
-    <link name="${name}_LS_link">
-      <inertial>
-        <origin xyz="-5.8187E-13 -0.062713 0" rpy="0 0 0" />
-        <mass value="${swivel_mass}" />
-        <inertia ixx="0.0010313" ixy="1.377E-13" ixz="1.6475E-20" iyy="0.00038801" iyz="2.1123E-20" izz="0.001103" />
-      </inertial>
-      <xacro:insert_block name="swivel_visual_collision" />
-    </link>
-    <xacro:wheel_joint joint_name="${name}_joint_LW" parent="${name}_LS_link" child="${name}_LW_link"
+      x="-0.32996" y="-0.1905" hardware_interface="${hardware_interface}"/>
+      <link name="${name}_LS_link">
+        <inertial>
+          <origin xyz="-5.8187E-13 -0.062713 0" rpy="0 0 0" />
+          <mass value="${swivel_mass}" />
+          <inertia ixx="0.0010313" ixy="1.377E-13" ixz="1.6475E-20" iyy="0.00038801" iyz="2.1123E-20" izz="0.001103" />
+        </inertial>
+        <xacro:insert_block name="swivel_visual_collision" />
+      </link>
+      <xacro:wheel_joint joint_name="${name}_joint_LW" parent="${name}_LS_link" child="${name}_LW_link"
         hardware_interface="${hardware_interface}"/>
-    <link name="${name}_LW_link">
-      <inertial>
-        <origin xyz="0 2.7756E-17 0" rpy="0 0 0" />
-        <mass value="${wheel_mass}" />
-        <inertia ixx="0.00016727" ixy="-1.3787E-22" ixz="-1.031E-22" iyy="9.626E-05" iyz="-3.3087E-21" izz="9.626E-05" />
-      </inertial>
-      <xacro:insert_block name="wheel_visual_collision" />
-    </link>
+        <link name="${name}_LW_link">
+          <inertial>
+            <origin xyz="0 2.7756E-17 0" rpy="0 0 0" />
+            <mass value="${wheel_mass}" />
+            <inertia ixx="0.00016727" ixy="-1.3787E-22" ixz="-1.031E-22" iyy="9.626E-05" iyz="-3.3087E-21" izz="9.626E-05" />
+          </inertial>
+          <xacro:insert_block name="wheel_visual_collision" />
+        </link>
     <!--
       RIGHT SWIVEL DEFINITION
     -->
     <xacro:swerve_joint joint_name="${name}_joint_RS" parent="${name}_body" child="${name}_RS_link"
-        x="0.32996" y="-0.1905"  hardware_interface="${hardware_interface}"/>
-    <link name="${name}_RS_link">
+      x="0.32996" y="-0.1905"  hardware_interface="${hardware_interface}"/>
+      <link name="${name}_RS_link">
+        <inertial>
+          <origin xyz="-5.8192E-13 -0.062713 -2.7756E-17" rpy="0 0 0" />
+          <mass value="${swivel_mass}" />
+          <inertia ixx="0.0010313" ixy="1.377E-13" ixz="1.6475E-20" iyy="0.00038801" iyz="2.1123E-20" izz="0.001103" />
+        </inertial>
+        <xacro:insert_block name="swivel_visual_collision" />
+      </link>
+      <xacro:wheel_joint joint_name="${name}_joint_RW" parent="${name}_RS_link" child="${name}_RW_link"
+        hardware_interface="${hardware_interface}"/>
+        <link name="${name}_RW_link">
+          <inertial>
+            <origin xyz="-5.5511E-17 2.7756E-17 -2.7756E-17" rpy="0 0 0" />
+            <mass value="${wheel_mass}" />
+            <inertia ixx="0.00016727" ixy="-1.3787E-22" ixz="-1.031E-22" iyy="9.626E-05" iyz="-3.3087E-21" izz="9.626E-05" />
+          </inertial>
+          <xacro:insert_block name="wheel_visual_collision" />
+        </link>
+    <!--
+      SENSORS
+    -->
+    <link name="laser">
+      <visual>
+        <origin xyz="0 0 0" rpy="0 0 0" />
+        <geometry>
+          <mesh filename="package://sick_tim/meshes/sick_tim551.stl" />
+        </geometry>
+        <xacro:insert_block name="color_blue" />
+      </visual>
       <inertial>
-        <origin xyz="-5.8192E-13 -0.062713 -2.7756E-17" rpy="0 0 0" />
-        <mass value="${swivel_mass}" />
-        <inertia ixx="0.0010313" ixy="1.377E-13" ixz="1.6475E-20" iyy="0.00038801" iyz="2.1123E-20" izz="0.001103" />
+        <mass value="0.001" />
+        <origin xyz="0 0 0" />
+        <inertia ixx="0.0001" ixy="0.0" ixz="0.0" iyy="0.0001" iyz="0.0" izz="0.0001" />
       </inertial>
-      <xacro:insert_block name="swivel_visual_collision" />
     </link>
-    <xacro:wheel_joint joint_name="${name}_joint_RW" parent="${name}_RS_link" child="${name}_RW_link"
-        hardware_interface="${hardware_interface}"/>
-    <link name="${name}_RW_link">
-      <inertial>
-        <origin xyz="-5.5511E-17 2.7756E-17 -2.7756E-17" rpy="0 0 0" />
-        <mass value="${wheel_mass}" />
-        <inertia ixx="0.00016727" ixy="-1.3787E-22" ixz="-1.031E-22" iyy="9.626E-05" iyz="-3.3087E-21" izz="9.626E-05" />
-      </inertial>
-      <xacro:insert_block name="wheel_visual_collision" />
+    <joint name="laser_joint" type="fixed">
+      <origin xyz="0 0.2 0.063" rpy="0 0 ${pi}" />
+      <parent link="${name}_body" />
+      <child link="laser" />
+    </joint>
+    <!-- from Stereo Labs: https://goo.gl/UvqS36 -->
+    <link name="zed_center">
+      <visual>
+        <origin xyz="0 0 0" rpy="0 0 0"/>
+        <geometry>
+          <mesh filename="package://swerve_description/meshes/ZED.stl" />
+        </geometry>
+        <material name="light_grey">
+          <color rgba="0.8 0.8 0.8 0.8"/>
+        </material>
+      </visual>
     </link>
+    <joint name="zed_camera_joint" type="fixed">
+      <parent link="${name}_body"/>
+      <child link="zed_center"/>
+      <origin xyz="0 0.18 0.11" rpy="0 0 ${pi}" />
+    </joint>
+    <link name="zed_left_camera">
+      <visual>
+        <origin xyz="0 0 0" rpy="0 ${pi} 0"/>
+        <geometry>
+          <cylinder radius="0.007" length=".031"/>
+        </geometry>
+        <material name="dark_grey">
+          <color rgba="0.1 0.1 0.1 1"/>
+        </material>
+      </visual>
+    </link>
+    <link name="zed_right_camera">
+      <visual>
+        <origin xyz="0 0 0" rpy="0 ${pi} 0"/>
+        <geometry>
+          <cylinder radius="0.007" length=".031"/>
+        </geometry>
+        <material name="dark_grey">
+          <color rgba="0.1 0.1 0.1 1"/>
+        </material>
+      </visual>
+    </link>
+    <joint name="zed_left_camera_joint" type="fixed">
+      <parent link="zed_center"/>
+      <child link="zed_left_camera"/>
+      <origin xyz="0.2 0.06 0" rpy="0 0 0" />
+    </joint>
+    <joint name="zed_right_camera_joint" type="fixed">
+      <parent link="zed_center"/>
+      <child link="zed_right_camera"/>
+      <origin xyz="0 -0.06 0" rpy="0 0 0" />
+    </joint>
+    <link name="zed_depth_camera" />
+    <joint name="zed_depth_camera_joint" type="fixed">
+      <parent link="zed_left_camera"/>
+      <child link="zed_depth_camera"/>
+      <origin xyz="0 0 0" rpy="-1.5707963267948966 0 -1.5707963267948966" />
+    </joint>
   </xacro:macro>
 </robot>

File: swerve_description/urdf/swerve_gazebo.xacro (robot description, xacro)
@@ -7,18 +7,222 @@
 -->
 <robot name="swerve" xmlns:xacro="http://www.ros.org/wiki/xacro">
-  <gazebo>
-    <plugin name="gazebo_ros_controller" filename="libgazebo_ros_control.so">
-      <robotNamespace>/swerve</robotNamespace>
-    </plugin>
-    <plugin name="p3d_base_controller" filename="libgazebo_ros_p3d.so">
-		  <alwaysOn>true</alwaysOn>
-		  <updateRate>50.0</updateRate>
-		  <bodyName>odom</bodyName>
-		  <topicName>odom</topicName>
-		  <gaussianNoise>0.01</gaussianNoise>
-		  <frameName>world</frameName>
-		  <xyzOffsets>0 0 0</xyzOffsets>
-		  <rpyOffsets>0 0 0</rpyOffsets>
+  <!--
+    ODOM CONTROLLER
+  -->
+	<gazebo>
+		<plugin name="gazebo_ros_controller" filename="libgazebo_ros_control.so">
+			<robotNamespace>/swerve</robotNamespace>
 		</plugin>
+		<plugin name="p3d_base_controller" filename="libgazebo_ros_p3d.so">
+			<alwaysOn>true</alwaysOn>
+			<updateRate>50.0</updateRate>
+			<bodyName>odom</bodyName>
+			<topicName>odom</topicName>
+			<gaussianNoise>0.01</gaussianNoise>
+			<frameName>world</frameName>
+			<xyzOffsets>0 0 0</xyzOffsets>
+			<rpyOffsets>0 0 0</rpyOffsets>
+		</plugin>
+	</gazebo>
+  <!--
+    LIDAR
+  -->
+	<gazebo reference="laser">
+    <sensor type="gpu_ray" name="laser">
+      <always_on>true</always_on>
+      <pose>0 0 0 0 0 0</pose>
+      <visualize>false</visualize>
+      <update_rate>15</update_rate>
+      <ray>
+        <scan>
+          <horizontal>
+            <samples>810</samples>
+            <resolution>1</resolution>
+            <min_angle>-2.35619</min_angle>
+            <max_angle>2.35619</max_angle>
+          </horizontal>
+        </scan>
+        <range>
+          <min>0.10</min>
+          <max>20.0</max>
+          <resolution>0.01</resolution>
+        </range>
+        <noise>
+          <type>gaussian</type>
+          <!-- Noise parameters based on published spec for Hokuyo laser
+               achieving "+-30mm" accuracy at range < 10m.  A mean of 0.0m and
+               stddev of 0.01m will put 99.7% of samples within 0.03m of the true
+               reading. -->
+          <mean>0.0</mean>
+          <stddev>0.01</stddev>
+        </noise>
+      </ray>
+      <plugin name="gazebo_ros_head_hokuyo_controller" filename="libgazebo_ros_gpu_laser.so">
+        <topicName>scan</topicName>
+        <frameName>laser</frameName>
+      </plugin>
+    </sensor>
   </gazebo>
+  <!--
+    ZED CAMERA
+  -->
+  <gazebo reference="zed_left_camera">
+    <material>Gazebo/Green</material>
+    <sensor type="camera" name="left_camera">
+      <update_rate>30.0</update_rate>
+      <camera name="left">
+        <horizontal_fov>2.0</horizontal_fov>
+        <image>
+          <width>800</width>
+          <height>800</height>
+          <format>R8G8B8</format>
+        </image>
+        <clip>
+          <near>0.02</near>
+          <far>300</far>
+        </clip>
+      </camera>
+      <plugin name="camera_controller" filename="libgazebo_ros_camera.so">
+        <alwaysOn>true</alwaysOn>
+        <updateRate>0.0</updateRate>
+        <cameraName>camera/left</cameraName>
+        <imageTopicName>image_raw</imageTopicName>
+        <cameraInfoTopicName>camera_info</cameraInfoTopicName>
+        <frameName>zed_left_camera</frameName>
+        <hackBaseline>0.07</hackBaseline>
+        <distortionK1>0.0</distortionK1>
+        <distortionK2>0.0</distortionK2>
+        <distortionK3>0.0</distortionK3>
+        <distortionT1>0.0</distortionT1>
+        <distortionT2>0.0</distortionT2>
+      </plugin>
+    </sensor>
+  </gazebo>
+  <!-- <gazebo reference="zed_left_camera">
+    <sensor type="camera" name="zed_left_camera">
+      <update_rate>30.0</update_rate>
+      <camera name="zed_left_camera">
+        <horizontal_fov>0.8709216071359963</horizontal_fov>
+        <image>
+          <width>640</width>
+          <height>480</height>
+          <format>B8G8R8</format>
+        </image>
+        <clip>
+          <near>0.02</near>
+          <far>300</far>
+        </clip>
+        <noise>
+          <type>gaussian</type>
+          <mean>0.0</mean>
+          <stddev>0.007</stddev>
+        </noise>
+      </camera>
+      <plugin name="camera_controller" filename="libgazebo_ros_camera.so">
+        <alwaysOn>true</alwaysOn>
+        <updateRate>30.0</updateRate>
+        <cameraName>/camera/left</cameraName>
+        <imageTopicName>image_raw_color</imageTopicName>
+        <cameraInfoTopicName>camera_info</cameraInfoTopicName>
+        <frameName>zed_left_camera</frameName>
+        <hackBaseline>0</hackBaseline>
+        <distortionK1>0.0</distortionK1>
+        <distortionK2>0.0</distortionK2>
+        <distortionK3>0.0</distortionK3>
+        <distortionT1>0.0</distortionT1>
+        <distortionT2>0.0</distortionT2>
+      </plugin>
+    </sensor>
+  </gazebo> -->
+  <!-- <gazebo reference="zed_right_camera">
+    <sensor type="camera" name="zed_right_camera">
+      <update_rate>30.0</update_rate>
+      <camera name="zed_right_camera">
+        <horizontal_fov>0.8709216071359963</horizontal_fov>
+        <image>
+          <width>640</width>
+          <height>480</height>
+          <format>B8G8R8</format>
+        </image>
+        <clip>
+          <near>0.02</near>
+          <far>300</far>
+        </clip>
+        <noise>
+          <type>gaussian</type>
+          <mean>0.0</mean>
+          <stddev>0.007</stddev>
+        </noise>
+      </camera>
+      <plugin name="camera_controller" filename="libgazebo_ros_camera.so">
+        <alwaysOn>true</alwaysOn>
+        <updateRate>30.0</updateRate>
+        <cameraName>/camera/right</cameraName>
+        <imageTopicName>image_raw_color</imageTopicName>
+        <cameraInfoTopicName>camera_info</cameraInfoTopicName>
+        <frameName>zed_right_camera</frameName>
+        <hackBaseline>0</hackBaseline>
+        <distortionK1>0.0</distortionK1>
+        <distortionK2>0.0</distortionK2>
+        <distortionK3>0.0</distortionK3>
+        <distortionT1>0.0</distortionT1>
+        <distortionT2>0.0</distortionT2>
+      </plugin>
+    </sensor>
+  </gazebo> -->
+  <!-- <gazebo reference="zed_center">
+    <sensor type="multicamera" name="zed_camera">
+      <update_rate>30.0</update_rate>
+      <camera name="zed_left_camera">
+        <pose>0 0.06 0 0 0 0</pose>
+        <horizontal_fov>0.8709216071359963</horizontal_fov>
+        <image>
+          <width>640</width>
+          <height>480</height>
+          <format>R8G8B8</format>
+        </image>
+        <clip>
+          <near>0.02</near>
+          <far>300</far>
+        </clip>
+        <noise>
+          <type>gaussian</type>
+          <mean>0.0</mean>
+          <stddev>0.007</stddev>
+        </noise>
+      </camera>
+      <camera name="zed_right_camera">
+        <pose>0 -0.06 0 0 0 0</pose>
+        <horizontal_fov>0.8709216071359963</horizontal_fov>
+        <image>
+          <width>640</width>
+          <height>480</height>
+          <format>R8G8B8</format>
+        </image>
+        <clip>
+          <near>0.02</near>
+          <far>300</far>
+        </clip>
+        <noise>
+          <type>gaussian</type>
+          <mean>0.0</mean>
+          <stddev>0.007</stddev>
+        </noise>
+      </camera>
+      <plugin name="stereo_camera_controller" filename="libgazebo_ros_multicamera.so">
+        <alwaysOn>true</alwaysOn>
+        <updateRate>0.0</updateRate>
+        <cameraName>camera</cameraName>
+        <imageTopicName>image_raw_color</imageTopicName>
+        <cameraInfoTopicName>camera_info</cameraInfoTopicName>
+        <frameName>zed_center</frameName>
+        <hackBaseline>0</hackBaseline>
+        <distortionK1>0.0</distortionK1>
+        <distortionK2>0.0</distortionK2>
+        <distortionK3>0.0</distortionK3>
+        <distortionT1>0.0</distortionT1>
+        <distortionT2>0.0</distortionT2>
+      </plugin>
+    </sensor>
+  </gazebo> -->
 </robot>

File: swerve_description/urdf/swerve_utilities.xacro (robot description, xacro)
@@ -8,4 +8,5 @@
 <robot name="swerve" xmlns:xacro="http://www.ros.org/wiki/xacro">
   <!-- Constants -->
+  <xacro:property name="pi" value="1.5708" />
   <xacro:property name="chassis_mass" value="7.0052" />
   <xacro:property name="swivel_mass" value="0.449039" />
