Commit message: Updated Swerve urdf to Kinetic standards

File: swerve_description/urdf/swerve.urdf.xacro (robot description, xacro)
@@ -26,5 +26,6 @@
   <!-- Define macros for swerve import -->
   <xacro:swerve name="swerve" parent="odom" hardware_interface="$(arg hardware_interface)">
-	  <origin xyz="0 0 0.17" rpy="0 0 -${pi}"/> <!-- rotate 90 degrees due to error in black box model -->
+	  <origin xyz="0 0 0.17" rpy="0 0 -${pi/2}"/> <!-- rotate 90 degrees due to error in black box model -->
   </xacro:swerve>
+  <xacro:swerve_sensors name="swerve"/>
 </robot>

File: swerve_description/urdf/swerve.xacro (robot description, xacro)
@@ -7,6 +7,4 @@
 -->
 <robot name="swerve" xmlns:xacro="http://www.ros.org/wiki/xacro">
-  <!-- Include constants and modeling macros -->
-  <xacro:include filename="$(find swerve_description)/urdf/swerve_utilities.xacro" />
   <xacro:macro name="swerve" params="parent name *origin hardware_interface">
     <!--
@@ -14,5 +12,5 @@
     -->
     <joint name="${parent}_joint" type="fixed">
-      <insert_block name="origin" />
+      <xacro:insert_block name="origin" />
       <parent link="${parent}" />
       <child link="${name}_body" />
@@ -44,12 +42,12 @@
     <xacro:wheel_joint joint_name="${name}_joint_FW" parent="${name}_FS_link" child="${name}_FW_link"
       hardware_interface="${hardware_interface}"/>
-      <link name="${name}_FW_link">
-        <inertial>
-          <origin xyz="-7.8185E-19 2.7756E-17 5.5511E-17" rpy="0 0 0" />
-          <mass value="${wheel_mass}" />
-          <inertia ixx="0.00016727" ixy="-4.9394E-22" ixz="-2.3462E-22" iyy="9.626E-05" iyz="-1.4682E-20" izz="9.626E-05" />
-        </inertial>
-        <xacro:insert_block name="wheel_visual_collision" />
-      </link>
+    <link name="${name}_FW_link">
+      <inertial>
+        <origin xyz="-7.8185E-19 2.7756E-17 5.5511E-17" rpy="0 0 0" />
+        <mass value="${wheel_mass}" />
+        <inertia ixx="0.00016727" ixy="-4.9394E-22" ixz="-2.3462E-22" iyy="9.626E-05" iyz="-1.4682E-20" izz="9.626E-05" />
+      </inertial>
+      <xacro:insert_block name="wheel_visual_collision" />
+    </link>
     <!--
       LEFT SWIVEL DEFINITION
@@ -67,12 +65,12 @@
     <xacro:wheel_joint joint_name="${name}_joint_LW" parent="${name}_LS_link" child="${name}_LW_link"
       hardware_interface="${hardware_interface}"/>
-      <link name="${name}_LW_link">
-        <inertial>
-          <origin xyz="0 2.7756E-17 0" rpy="0 0 0" />
-          <mass value="${wheel_mass}" />
-          <inertia ixx="0.00016727" ixy="-1.3787E-22" ixz="-1.031E-22" iyy="9.626E-05" iyz="-3.3087E-21" izz="9.626E-05" />
-        </inertial>
-        <xacro:insert_block name="wheel_visual_collision" />
-      </link>
+    <link name="${name}_LW_link">
+      <inertial>
+        <origin xyz="0 2.7756E-17 0" rpy="0 0 0" />
+        <mass value="${wheel_mass}" />
+        <inertia ixx="0.00016727" ixy="-1.3787E-22" ixz="-1.031E-22" iyy="9.626E-05" iyz="-3.3087E-21" izz="9.626E-05" />
+      </inertial>
+      <xacro:insert_block name="wheel_visual_collision" />
+    </link>
     <!--
       RIGHT SWIVEL DEFINITION
@@ -90,16 +88,16 @@
     <xacro:wheel_joint joint_name="${name}_joint_RW" parent="${name}_RS_link" child="${name}_RW_link"
       hardware_interface="${hardware_interface}"/>
-      <link name="${name}_RW_link">
-        <inertial>
-          <origin xyz="-5.5511E-17 2.7756E-17 -2.7756E-17" rpy="0 0 0" />
-          <mass value="${wheel_mass}" />
-          <inertia ixx="0.00016727" ixy="-1.3787E-22" ixz="-1.031E-22" iyy="9.626E-05" iyz="-3.3087E-21" izz="9.626E-05" />
-        </inertial>
-        <xacro:insert_block name="wheel_visual_collision" />
-      </link>
+    <link name="${name}_RW_link">
+      <inertial>
+        <origin xyz="-5.5511E-17 2.7756E-17 -2.7756E-17" rpy="0 0 0" />
+        <mass value="${wheel_mass}" />
+        <inertia ixx="0.00016727" ixy="-1.3787E-22" ixz="-1.031E-22" iyy="9.626E-05" iyz="-3.3087E-21" izz="9.626E-05" />
+      </inertial>
+      <xacro:insert_block name="wheel_visual_collision" />
+    </link>
     <!--
       SENSORS
     -->
-    <link name="laser">
+    <link name="${name}_laser">
       <visual>
         <origin xyz="0 0 0" rpy="0 0 0" />
@@ -115,11 +113,11 @@
       </inertial>
     </link>
-    <joint name="laser_joint" type="fixed">
-      <origin xyz="0 0.2 0.063" rpy="0 0 ${pi}" />
+    <joint name="${name}_laser_joint" type="fixed">
+      <origin xyz="0 0.2 0.063" rpy="0 0 ${pi/2}" />
       <parent link="${name}_body" />
-      <child link="laser" />
+      <child link="${name}_laser" />
     </joint>
     <!-- from Stereo Labs: https://goo.gl/UvqS36 -->
-    <link name="zed_center">
+    <link name="${name}_zed_center">
       <visual>
         <origin xyz="0 0 0" rpy="0 0 0"/>
@@ -134,14 +132,14 @@
     <joint name="zed_camera_joint" type="fixed">
       <parent link="${name}_body"/>
-      <child link="zed_center"/>
-      <origin xyz="0 0.18 0.11" rpy="0 0 ${pi}" />
+      <child link="${name}_zed_center"/>
+      <origin xyz="0 0.18 0.11" rpy="0 0 ${pi/2}" />
     </joint>
-    <link name="zed_depth"></link>
-    <joint name="zed_depth_joint" type="fixed">
-      <parent link="zed_center"/>
-      <child link="zed_depth"/>
+    <link name="${name}_zed_depth"></link>
+    <joint name="${name}_zed_depth_joint" type="fixed">
+      <parent link="${name}_zed_center"/>
+      <child link="${name}_zed_depth"/>
       <origin xyz="0 0 0" rpy="${pi} 0 ${pi}" />
     </joint>
-    <link name="zed_left_camera">
+    <link name="${name}_zed_left_camera">
       <visual>
         <origin xyz="0 0 0" rpy="0 ${pi} 0"/>
@@ -154,5 +152,5 @@
       </visual>
     </link>
-    <link name="zed_right_camera">
+    <link name="${name}_zed_right_camera">
       <visual>
         <origin xyz="0 0 0" rpy="0 ${pi} 0"/>
@@ -165,18 +163,18 @@
       </visual>
     </link>
-    <joint name="zed_left_camera_joint" type="fixed">
-      <parent link="zed_center"/>
-      <child link="zed_left_camera"/>
+    <joint name="${name}_zed_left_camera_joint" type="fixed">
+      <parent link="${name}_zed_center"/>
+      <child link="${name}_zed_left_camera"/>
       <origin xyz="0 0.06 0" rpy="0 0 0" />
     </joint>
-    <joint name="zed_right_camera_joint" type="fixed">
-      <parent link="zed_center"/>
-      <child link="zed_right_camera"/>
+    <joint name="${name}_zed_right_camera_joint" type="fixed">
+      <parent link="${name}_zed_center"/>
+      <child link="${name}_zed_right_camera"/>
       <origin xyz="0 -0.06 0" rpy="0 0 0" />
     </joint>
-    <link name="zed_depth_camera" />
-    <joint name="zed_depth_camera_joint" type="fixed">
-      <parent link="zed_left_camera"/>
-      <child link="zed_depth_camera"/>
+    <link name="${name}_zed_depth_camera" />
+    <joint name="${name}_zed_depth_camera_joint" type="fixed">
+      <parent link="${name}_zed_left_camera"/>
+      <child link="${name}_zed_depth_camera"/>
       <origin xyz="0 0 0" rpy="-1.5707963267948966 0 -1.5707963267948966" />
     </joint>

File: swerve_description/urdf/swerve_gazebo.xacro (robot description, xacro)
@@ -25,132 +25,134 @@
     </plugin>
   </gazebo>
-  <!--
-  LIDAR
-  -->
-  <gazebo reference="laser">
-    <sensor type="ray" name="laser">
-      <always_on>true</always_on>
-      <pose>0 0 0 0 0 0</pose>
-      <visualize>true</visualize>
-      <update_rate>15</update_rate>
-      <ray>
-        <scan>
-          <horizontal>
-            <samples>810</samples>
-            <resolution>1</resolution>
-            <min_angle>-2.35619</min_angle>
-            <max_angle>2.35619</max_angle>
-          </horizontal>
-        </scan>
-        <range>
-          <min>0.10</min>
-          <max>10.0</max>
-          <resolution>0.01</resolution>
-        </range>
-        <noise>
-          <type>gaussian</type>
-           <mean>0.0</mean>
-           <stddev>0.00667</stddev>
-         </noise>
-       </ray>
-       <plugin name="gazebo_ros_head_hokuyo_controller" filename="libgazebo_ros_laser.so">
-        <topicName>scan</topicName>
-        <frameName>laser</frameName>
-      </plugin>
-    </sensor>
-  </gazebo>
-  <!--
-  ZED CAMERA
-  -->
-  <!--<gazebo reference="zed_center">
-    <sensor type="multicamera" name="zed_camera">
-      <update_rate>30.0</update_rate>
-      <camera name="zed_left_camera">
-        <pose>0 0.06 0 0 0 0</pose>
-        <horizontal_fov>0.8709216071359963</horizontal_fov>
-        <image>
-          <width>640</width>
-          <height>480</height>
-          <format>R8G8B8</format>
-        </image>
-        <clip>
-          <near>0.5</near>
-          <far>20</far>
-        </clip>
-        <noise>
-          <type>gaussian</type>
-          <mean>0.0</mean>
-          <stddev>0.007</stddev>
-        </noise>
-      </camera>
-      <camera name="zed_right_camera">
-        <pose>0 -0.06 0 0 0 0</pose>
-        <horizontal_fov>0.8709216071359963</horizontal_fov>
-        <image>
-          <width>640</width>
-          <height>480</height>
-          <format>R8G8B8</format>
-        </image>
-        <clip>
-          <near>0.5</near>
-          <far>20</far>
-        </clip>
-        <noise>
-          <type>gaussian</type>
-          <mean>0.0</mean>
-          <stddev>0.007</stddev>
-        </noise>
-      </camera>
-      <plugin name="stereo_camera_controller" filename="libgazebo_ros_multicamera.so">
-        <alwaysOn>true</alwaysOn>
-        <updateRate>0.0</updateRate>
-        <cameraName>camera</cameraName>
-        <imageTopicName>image_raw</imageTopicName>
-        <cameraInfoTopicName>camera_info</cameraInfoTopicName>
-        <frameName>zed_center</frameName>
-        <hackBaseline>0</hackBaseline>
-        <distortionK1>0.0</distortionK1>
-        <distortionK2>0.0</distortionK2>
-        <distortionK3>0.0</distortionK3>
-        <distortionT1>0.0</distortionT1>
-        <distortionT2>0.0</distortionT2>
-      </plugin>
-    </sensor>
-  </gazebo>
-  <gazebo reference="zed_depth">
-    <sensor type="depth" name="camera">
-      <always_on>true</always_on>
-      <update_rate>20.0</update_rate>
-      <camera>
-        <horizontal_fov>2.0</horizontal_fov>
-        <image>
-          <format>B8G8R8</format>
-          <width>640</width>
-          <height>480</height>
-        </image>
-        <clip>
-          <near>0.05</near>
-          <far>8.0</far>
-        </clip>
-      </camera>
-      <plugin name="kinect_camera_controller" filename="libgazebo_ros_openni_kinect.so">
-        <cameraName>camera</cameraName>
-        <alwaysOn>true</alwaysOn>
-        <updateRate>10</updateRate>
-        <imageTopicName>rgb/image_raw</imageTopicName>
-        <depthImageTopicName>depth/image_raw</depthImageTopicName>
-        <pointCloudTopicName>depth/points</pointCloudTopicName>
-        <cameraInfoTopicName>rgb/camera_info</cameraInfoTopicName>
-        <depthImageCameraInfoTopicName>depth/camera_info</depthImageCameraInfoTopicName>
-        <frameName>zed_depth</frameName>
-        <baseline>0.1</baseline>
-        <distortion_k1>0.0</distortion_k1>
-        <distortion_k2>0.0</distortion_k2>
-        <distortion_k3>0.0</distortion_k3>
-        <distortion_t1>0.0</distortion_t1>
-        <distortion_t2>0.0</distortion_t2>
-        <pointCloudCutoff>0.4</pointCloudCutoff>
-      </plugin>
-    </sensor>
-  </gazebo>-->
+  <xacro:macro name="swerve_sensors" params="name">
+    <!--
+    LIDAR
+    -->
+    <gazebo reference="${name}_laser">
+      <sensor type="ray" name="${name}_laser">
+        <always_on>true</always_on>
+        <pose>0 0 0 0 0 0</pose>
+        <visualize>true</visualize>
+        <update_rate>15</update_rate>
+        <ray>
+          <scan>
+            <horizontal>
+              <samples>810</samples>
+              <resolution>1</resolution>
+              <min_angle>-2.35619</min_angle>
+              <max_angle>2.35619</max_angle>
+            </horizontal>
+          </scan>
+          <range>
+            <min>0.10</min>
+            <max>10.0</max>
+            <resolution>0.01</resolution>
+          </range>
+          <noise>
+            <type>gaussian</type>
+             <mean>0.0</mean>
+             <stddev>0.00667</stddev>
+           </noise>
+         </ray>
+         <plugin name="gazebo_ros_head_hokuyo_controller" filename="libgazebo_ros_laser.so">
+          <topicName>scan</topicName>
+          <frameName>${name}_laser</frameName>
+        </plugin>
+      </sensor>
+    </gazebo>
+    <!--
+    ZED CAMERA
+    -->
+    <!--<gazebo reference="${name}_zed_center">
+      <sensor type="multicamera" name="${name}_zed_camera">
+        <update_rate>30.0</update_rate>
+        <camera name="${name}_zed_left_camera">
+          <pose>0 0.06 0 0 0 0</pose>
+          <horizontal_fov>0.8709216071359963</horizontal_fov>
+          <image>
+            <width>640</width>
+            <height>480</height>
+            <format>R8G8B8</format>
+          </image>
+          <clip>
+            <near>0.5</near>
+            <far>20</far>
+          </clip>
+          <noise>
+            <type>gaussian</type>
+            <mean>0.0</mean>
+            <stddev>0.007</stddev>
+          </noise>
+        </camera>
+        <camera name="${name}_zed_right_camera">
+          <pose>0 -0.06 0 0 0 0</pose>
+          <horizontal_fov>0.8709216071359963</horizontal_fov>
+          <image>
+            <width>640</width>
+            <height>480</height>
+            <format>R8G8B8</format>
+          </image>
+          <clip>
+            <near>0.5</near>
+            <far>20</far>
+          </clip>
+          <noise>
+            <type>gaussian</type>
+            <mean>0.0</mean>
+            <stddev>0.007</stddev>
+          </noise>
+        </camera>
+        <plugin name="${name}_stereo_camera_controller" filename="libgazebo_ros_multicamera.so">
+          <alwaysOn>true</alwaysOn>
+          <updateRate>0.0</updateRate>
+          <cameraName>camera</cameraName>
+          <imageTopicName>image_raw</imageTopicName>
+          <cameraInfoTopicName>camera_info</cameraInfoTopicName>
+          <frameName>${name}_zed_center</frameName>
+          <hackBaseline>0</hackBaseline>
+          <distortionK1>0.0</distortionK1>
+          <distortionK2>0.0</distortionK2>
+          <distortionK3>0.0</distortionK3>
+          <distortionT1>0.0</distortionT1>
+          <distortionT2>0.0</distortionT2>
+        </plugin>
+      </sensor>
+    </gazebo>
+    <gazebo reference="${name}_zed_depth">
+      <sensor type="depth" name="camera">
+        <always_on>true</always_on>
+        <update_rate>20.0</update_rate>
+        <camera>
+          <horizontal_fov>2.0</horizontal_fov>
+          <image>
+            <format>B8G8R8</format>
+            <width>640</width>
+            <height>480</height>
+          </image>
+          <clip>
+            <near>0.05</near>
+            <far>8.0</far>
+          </clip>
+        </camera>
+        <plugin name="${name}_kinect_camera_controller" filename="libgazebo_ros_openni_kinect.so">
+          <cameraName>camera</cameraName>
+          <alwaysOn>true</alwaysOn>
+          <updateRate>10</updateRate>
+          <imageTopicName>rgb/image_raw</imageTopicName>
+          <depthImageTopicName>depth/image_raw</depthImageTopicName>
+          <pointCloudTopicName>depth/points</pointCloudTopicName>
+          <cameraInfoTopicName>rgb/camera_info</cameraInfoTopicName>
+          <depthImageCameraInfoTopicName>depth/camera_info</depthImageCameraInfoTopicName>
+          <frameName>${name}_zed_depth</frameName>
+          <baseline>0.1</baseline>
+          <distortion_k1>0.0</distortion_k1>
+          <distortion_k2>0.0</distortion_k2>
+          <distortion_k3>0.0</distortion_k3>
+          <distortion_t1>0.0</distortion_t1>
+          <distortion_t2>0.0</distortion_t2>
+          <pointCloudCutoff>0.4</pointCloudCutoff>
+        </plugin>
+      </sensor>
+    </gazebo>-->
+  </xacro:macro>
 </robot>

File: swerve_description/urdf/swerve_utilities.xacro (robot description, xacro)
@@ -8,5 +8,4 @@
 <robot name="swerve" xmlns:xacro="http://www.ros.org/wiki/xacro">
   <!-- Constants -->
-  <xacro:property name="pi" value="1.5708" />
   <xacro:property name="chassis_mass" value="7.0052" />
   <xacro:property name="swivel_mass" value="0.449039" />

Commit message: Development on Gazebo swerve

File: swerve_description/urdf/swerve.urdf.xacro (robot description, xacro)
@@ -25,5 +25,5 @@
   -->
   <!-- Define macros for swerve import -->
-  <xacro:swerve name="swerve" parent="odom" hardware_interface="$(arg hardware_interface)">
+  <xacro:swerve name="$(arg robot_name)" parent="odom" hardware_interface="$(arg hardware_interface)">
 	  <origin xyz="0 0 0.17" rpy="0 0 -${pi/2}"/> <!-- rotate 90 degrees due to error in black box model -->
   </xacro:swerve>

File: swerve_description/urdf/swerve.xacro (robot description, xacro)
@@ -139,5 +139,5 @@
       <parent link="${name}_zed_center"/>
       <child link="${name}_zed_depth"/>
-      <origin xyz="0 0 0" rpy="${pi} 0 ${pi}" />
+      <origin xyz="0 0 0" rpy="0 ${pi/2} 0" />
     </joint>
     <link name="${name}_zed_left_camera">

File: swerve_description/urdf/swerve_gazebo.xacro (robot description, xacro)
@@ -33,5 +33,5 @@
         <always_on>true</always_on>
         <pose>0 0 0 0 0 0</pose>
-        <visualize>true</visualize>
+        <visualize>false</visualize>
         <update_rate>15</update_rate>
         <ray>
@@ -64,5 +64,5 @@
     ZED CAMERA
     -->
-    <!--<gazebo reference="${name}_zed_center">
+    <gazebo reference="${name}_zed_center">
       <sensor type="multicamera" name="${name}_zed_camera">
         <update_rate>100.0</update_rate>
@@ -126,7 +126,7 @@
           <horizontal_fov>1.91986</horizontal_fov>
           <image>
-            <format>B8G8R8</format>
-            <width>640</width>
-            <height>480</height>
+            <width>2208</width>
+            <height>1242</height>
+            <format>R8G8B8</format>
           </image>
           <clip>
@@ -138,5 +138,5 @@
           <cameraName>camera</cameraName>
           <alwaysOn>true</alwaysOn>
-          <updateRate>10</updateRate>
+          <updateRate>10.0</updateRate>
           <imageTopicName>rgb/image_raw</imageTopicName>
           <depthImageTopicName>depth/image_raw</depthImageTopicName>
@@ -154,5 +154,5 @@
         </plugin>
       </sensor>
-    </gazebo>-->
+    </gazebo>
   </xacro:macro>
 </robot>
